File: nuco-v-kibot-test.kicad_pcb (KiCad board)
At the start: 2 copper layers, 70 x 82.5 mm, 141 parts, among them Q1 1N7002, Q2 1N7002, Q3 NTS4173, Q4 NTS4173, SW1 BUTTON1, SW2 BUTTON1, SW3 BUTTON1, U1 STM32H742Vx, U10 LP2985N, U2 LM1117, U3 LD39050PU, U4 SN74LVC2T45, U5 SN74LVC2T45, U6 SN74LVC2T45, U7 SN74LVC2T45, U8 ESDA5V3SC6, U9 STM32F103CBT6, X1 ST-MORPHO-CN7, X10 CONN-12P2L, X11 CONN-10P2L, X12 CONN-02P1LA, X13 CONN-02P1LA, X14 CONN-06P1L, X15 CONN-02P1L, X2 CONN-08P1L, X3 CONN-06P1L, X4 CONN-03P1L, X5 CONN-10P1L, X6 CONN-08P1L, X7 ST-MORPHO-CN10, X8 USB-OTG, X9 CONN-04P1L, Y1 32.768K, Y2 8MHz, Y3 8MHz

Commit message: Adds version and date flags
Other:
- board text added: "Version: %%version%% Date: %%date%%"
Changed lines of the file:
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@@
-(kicad_pcb (version 20171130) (host pcbnew 5.1.8-db9833491~87~ubuntu18.04.1)
+(kicad_pcb (version 20171130) (host pcbnew "(5.1.5)-3")
   (general
     (thickness 1.6)
-    (drawings 181)
+    (drawings 182)
     (tracks 2035)
     (zones 0)
@@
     (aux_axis_origin 70 140)
     (grid_origin 70 140)
-    (visible_elements FFFFFF7F)
+    (visible_elements 7FFFFFFF)
     (pcbplotparams
       (layerselection 0x010f0_ffffffff)
@@
     )
   )
+  (gr_text "Version: %%version%%\nDate: %%date%%" (at 127 140) (layer F.SilkS)
+    (effects (font (size 1 1) (thickness 0.15)))
+  )
   (gr_text GND (at 88.3 62.6) (layer F.SilkS)
